File: keychron-optical-keyboard.kicad_pcb (KiCad board)
At the start: 2 copper layers, 32.5 x 10 mm, 188 parts, among them U1 BlackPill_STLINK

Commit message: Route tracks, add switch plate, scripts
Add python scripts to route tracks, draw border, place footprints

A  Footprints.pretty/BlackPill_STLINK_Down.kicad_mod
A  Footprints.pretty/Border_PCB_WR.kicad_mod
M  Footprints.pretty/Keychron_Optical_Switch_1.25u.kicad_mod
M  Footprints.pretty/Keychron_Optical_Switch_1.5u.kicad_mod
D  Footprints.pretty/Keychron_Optical_Switch_1.75u.kicad_mod
M  Footprints.pretty/Keychron_Optical_Switch_1u.kicad_mod
D  Footprints.pretty/Keychron_Optical_Switch_2u.kicad_mod
A  Footprints.pretty/MountingHole_2.2mm_M2_ISO7380_Pad.kicad_mod
A  Footprints.pretty/SMTSO_M1.6.kicad_mod
A  Footprints.pretty/SMTSO_M2.kicad_mod
M  Footprints.pretty/Switch_Cutout.kicad_mod
M  MySymbols.kicad_sym
D  keychron-optical-keyboard-backups/keychron-optical-keyboard-2022-08-03_203051.zip
D  keychron-optical-keyboard-backups/keychron-optical-keyboard-2022-08-03_203709.zip
D  keychron-optical-keyboard-backups/keychron-optical-keyboard-2022-08-03_204429.zip
D  keychron-optical-keyboard-backups/keychron-optical-keyboard-2022-08-03_204938.zip
M  keychron-optical-keyboard.kicad_pcb
M  keychron-optical-keyboard.kicad_prl
M  keychron-optical-keyboard.kicad_sch
M  placek.py
A  resources/AL-S0602IRC-VI-12P9.pdf
A  resources/AL-S0602PTB-VI-1216.pdf
A  resources/IMG_0621.JPG
M  resources/keychronpic.png
A  switch-plate/.gitignore
A  switch-plate/fp-lib-table
A  switch-plate/switch-plate.kicad_pcb
A  switch-plate/switch-plate.kicad_prl
A  switch-plate/switch-plate.kicad_pro
A  switch-plate/switch-plate.kicad_sch
A  switch-plate/sym-lib-table
Parts:
- removed H18, H19, H20: MountingHole, MyFootprints:MountingHole_1.2mm_M1
- removed RL75: R_LED, Resistor_SMD:R_1206_3216Metric_Pad1.30x1.75mm_HandSolder
- removed S75: OptSw, MyFootprints:Keychron_Optical_Switch_1u
- removed TP1, TP2: TestPoint, TestPoint:TestPoint_THTPad_1.0x1.0mm_Drill0.5mm
- added D1: LED, LED_SMD:LED_0603_1608Metric_Pad1.05x0.95mm_HandSolder, F.Cu at (52.2, 71.2)
- added HS1: MountingHoleSprt, MyFootprints:SMTSO_M2, F.Cu at (-12.8, 168.5)
- added HS2: MountingHoleSprt, MyFootprints:SMTSO_M2, F.Cu at (69.8, 168.5)
- added HS3: MountingHoleSprt, MyFootprints:SMTSO_M2, F.Cu at (-12.8, 117.5)
- added HS4: MountingHoleSprt, MyFootprints:SMTSO_M2, F.Cu at (69.8, 117.5)
- added HS5: MountingHoleSprt, MyFootprints:SMTSO_M2, F.Cu at (205.8, 168.5)
- added HS6: MountingHoleSprt, MyFootprints:SMTSO_M2, F.Cu at (288.2, 168.5)
- added HS7: MountingHoleSprt, MyFootprints:SMTSO_M2, F.Cu at (205.8, 117.5)
- added HS8: MountingHoleSprt, MyFootprints:SMTSO_M2, F.Cu at (288.2, 117.5)
- added R1: R, Resistor_SMD:R_0805_2012Metric_Pad1.20x1.40mm_HandSolder, F.Cu at (60.5, 81.0)
- H1, H10, H11, H12, H13, H14, H15, H16, H2, H3, H4, H5, H6, H7, H8, H9: footprint MyFootprints:MountingHole_2.2mm_M2_jlcpcb -> MyFootprints:SMTSO_M1.6
- H17: footprint MyFootprints:MountingHole_1.2mm_M1 -> MyFootprints:SMTSO_M1.6
- RL1, RL10, RL11, RL12, RL13, RL14, RL15, RL16, RL17, RL18, RL19, RL2, RL20, RL21, RL22, RL23, RL24, RL25, RL26, RL27, RL28, RL29, RL3, RL30, RL31, RL32, RL33, RL34, RL35, RL36, RL37, RL38, RL39, RL4, RL40, RL41, RL42, RL43, RL44, RL45, RL46, RL47, RL48, RL49, RL5, RL50, RL51, RL52, RL53, RL54, RL55, RL56, RL57, RL58, RL59, RL6, RL60, RL61, RL62, RL63, RL64, RL65, RL66, RL67, RL68, RL69, RL7, RL70, RL71, RL72, RL73, RL74, RL8, RL9: value R_LED -> R_IR; footprint Resistor_SMD:R_1206_3216Metric_Pad1.30x1.75mm_HandSolder -> Resistor_SMD:R_0805_2012Metric_Pad1.20x1.40mm_HandSolder
- S32, S58: footprint MyFootprints:Keychron_Optical_Switch_1.25u -> MyFootprints:Keychron_Optical_Switch_1u
- S43, S45, S57, S64, S65, S67: footprint MyFootprints:Keychron_Optical_Switch_1u -> MyFootprints:Keychron_Optical_Switch_1.25u
- S44, S46, S66, S68: footprint MyFootprints:Keychron_Optical_Switch_1.75u -> MyFootprints:Keychron_Optical_Switch_1u
- U1: footprint MyFootprints:BlackPill_STLINK2 -> MyFootprints:BlackPill_STLINK_Down
- moved S30 282.8 mm to (14.2, 38.0)
- moved RL30 282.7 mm to (22.6, 36.5)
- moved S60 280.9 mm to (14.2, 76.0)
- moved RL60 280.9 mm to (22.6, 74.5)
- moved H1 278.7 mm to (9.50, -9.50)
- moved S45 273.8 mm to (21.4, 57.0)
- moved RL45 273.8 mm to (29.7, 55.5)
- moved H5 265.2 mm to (57.0, 10.1)
- moved H12 254.3 mm to (304.0, 48.1)
- moved RP1 244.8 mm to (13.1, 49.6), turned to 90 degrees
- moved RP2 221.4 mm to (34.5, 49.6), turned to 90 degrees
- moved RP5 220.0 mm to (91.5, 49.6), turned to 90 degrees
- moved H13 215.3 mm to (23.8, 85.5)
- moved RP3 211.9 mm to (53.5, 49.6), turned to 90 degrees
- moved H2 211.9 mm to (104.5, -9.50)
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Connections:
- RL30 pad 1: /row2 -> /row3
- RL45 pad 1: /row3 -> /row4
- RL60 pad 1: /row4 -> /row5
- S30 pad 3: /col15 -> /col1
- S31 pad 3: /col1 -> /col2
- S32 pad 3: /col2 -> /col3
- S33 pad 3: /col3 -> /col4
- S34 pad 3: /col4 -> /col5
- S35 pad 3: /col5 -> /col6
- S36 pad 3: /col6 -> /col7
- S37 pad 3: /col7 -> /col8
- S38 pad 3: /col8 -> /col9
- S39 pad 3: /col9 -> /col10
- S40 pad 3: /col10 -> /col11
- S41 pad 3: /col11 -> /col12
- S42 pad 3: /col12 -> /col13
- S43 pad 3: /col13 -> /col14
- S44 pad 3: /col14 -> /col15
- S45 pad 3: /col15 -> /col1
- S46 pad 3: /col1 -> /col2
- S47 pad 3: /col2 -> /col3
- S48 pad 3: /col3 -> /col4
- S49 pad 3: /col4 -> /col5
- S50 pad 3: /col5 -> /col6
- S51 pad 3: /col6 -> /col7
- S52 pad 3: /col7 -> /col8
- S53 pad 3: /col8 -> /col9
- S54 pad 3: /col9 -> /col10
- S55 pad 3: /col10 -> /col11
- S56 pad 3: /col11 -> /col12
- S57 pad 3: /col12 -> /col13
- S58 pad 3: /col13 -> /col14
- S59 pad 3: /col14 -> /col15
- S60 pad 3: /col15 -> /col1
- S61 pad 3: /col1 -> /col2
- S62 pad 3: /col2 -> /col3
- S63 pad 3: /col3 -> /col4
- S64 pad 3: /col4 -> /col5
- S65 pad 3: /col5 -> /col6
- S66 pad 3: /col6 -> /col7
- S67 pad 3: /col7 -> /col8
- S68 pad 3: /col8 -> /col9
- S69 pad 3: /col9 -> /col10
- S70 pad 3: /col10 -> /col11
- S71 pad 3: /col11 -> /col12
- S72 pad 3: /col12 -> /col13
- S73 pad 3: /col13 -> /col14
- S74 pad 3: /col14 -> /col15
Routing:
- net /col12: track 0.00 -> 450.6 mm, vias 0 -> 9
- net /col14: track 0.00 -> 443.4 mm, vias 0 -> 7
- net /col11: track 0.00 -> 434.3 mm, vias 0 -> 8
- net /col10: track 0.00 -> 414.9 mm, vias 0 -> 8
- net /col13: track 0.00 -> 411.9 mm, vias 0 -> 6
- net /col15: track 0.00 -> 392.7 mm, vias 0 -> 6
- net /col9: track 0.00 -> 384.3 mm, vias 0 -> 8
- net /col8: track 0.00 -> 375.0 mm, vias 0 -> 9
- net /row1: track 0.00 -> 360.3 mm, vias 0 -> 2
- net /col7: track 0.00 -> 351.4 mm, vias 0 -> 6
- net /col6: track 0.00 -> 327.2 mm, vias 0 -> 6
- net /row5: track 0.00 -> 326.3 mm, vias 0 -> 2
- net 3v3: track 0.00 -> 320.8 mm, vias 0 -> 1
- net /row2: track 0.00 -> 316.4 mm, vias 0 -> 2
- net /row4: track 0.00 -> 307.3 mm
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- added copper zone on B.Cu, net GND
Other:
- board size 32.5 x 10 mm -> 324.8 x 186 mm

Commit message: Add wrist support plate and remove 2 keys
A  Footprints.pretty/Keychron_Optical_Switch_1.75u.kicad_mod
A  drawborderk.py
M  keychron-optical-keyboard.kicad_pcb
M  keychron-optical-keyboard.kicad_prl
M  keychron-optical-keyboard.kicad_pro
M  keychron-optical-keyboard.kicad_sch
M  placek.py
M  switch-plate/switch-plate.kicad_pcb
M  switch-plate/switch-plate.kicad_sch
A  wrist-support/.gitignore
A  wrist-support/fp-lib-table
A  wrist-support/sym-lib-table
A  wrist-support/wrist-support.kicad_pcb
A  wrist-support/wrist-support.kicad_prl
A  wrist-support/wrist-support.kicad_pro
A  wrist-support/wrist-support.kicad_sch
Parts:
- removed RL73, RL74: R_IR, Resistor_SMD:R_0805_2012Metric_Pad1.20x1.40mm_HandSolder
- removed S73, S74: OptSw, MyFootprints:Keychron_Optical_Switch_1u
- S45: footprint MyFootprints:Keychron_Optical_Switch_1.25u -> MyFootprints:Keychron_Optical_Switch_1.5u
- S63, S66: footprint MyFootprints:Keychron_Optical_Switch_1u -> MyFootprints:Keychron_Optical_Switch_1.25u
- S65, S67: footprint MyFootprints:Keychron_Optical_Switch_1.25u -> MyFootprints:Keychron_Optical_Switch_1u
- moved RL59 280.9 mm to (22.6, 74.5)
- moved S59 280.9 mm to (14.2, 76.0)
- moved D1 69.2 mm to (118.8, 52.2)
- moved R1 69.2 mm to (127.0, 62.0)
- moved RL65 33.1 mm to (146.1, 74.5), turned to -90 degrees
- moved S65 29.7 mm to (137.8, 76.0), turned to 0 degrees
- moved S66 29.7 mm to (162.5, 92.5), turned to 110 degrees
- moved RL67 29.5 mm to (186.7, 77.3), turned to -74 degrees
- moved RL63 24.0 mm to (102.4, 81.8), turned to -106 degrees
- moved S63 23.3 mm to (94.0, 81.0), turned to -16 degrees
- moved S64 22.2 mm to (113.0, 92.5), turned to 70 degrees
- moved RL68 21.3 mm to (207.8, 74.5), turned to -90 degrees
- moved S68 21.0 mm to (199.5, 76.0), turned to 0 degrees
- moved S67 20.2 mm to (179.1, 81.0), turned to 16 degrees
- moved RL61 19.0 mm to (60.5, 74.5)
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Connections:
- RL59 pad 1: /row4 -> /row5
- S59 pad 3: /col15 -> /col1
- S60 pad 3: /col1 -> /col2
- S61 pad 3: /col2 -> /col3
- S62 pad 3: /col3 -> /col4
- S63 pad 3: /col4 -> /col5
- S64 pad 3: /col5 -> /col6
- S65 pad 3: /col6 -> /col7
- S66 pad 3: /col7 -> /col8
- S67 pad 3: /col8 -> /col9
- S68 pad 3: /col9 -> /col10
- S69 pad 3: /col10 -> /col11
- S70 pad 3: /col11 -> /col12
- S71 pad 3: /col12 -> /col13
- S72 pad 3: /col13 -> /col14
Routing:
- net /Capslock_Led: track 70.9 -> 130.4 mm, vias 1 -> 2
- net /col15: track 392.7 -> 340.3 mm, vias 6 -> 4
- net /col3: track 193.7 -> 213.3 mm
- net /row5: track 326.3 -> 310.8 mm, vias 2 -> 1
- net /row4: track 307.3 -> 292.5 mm
- net Net-(RL74-Pad2): track 11.8 -> 0.00 mm
- net Net-(RL73-Pad2): track 11.8 -> 0.00 mm
- net /col2: track 177.4 -> 183.3 mm
- net /col1: track 215.0 -> 209.6 mm
- net GND: track 205.2 -> 200.1 mm, vias 149 -> 145
- net Net-(RL68-Pad2): track 7.10 -> 11.8 mm
- net Net-(RL66-Pad2): track 11.8 -> 7.29 mm
- net Net-(RL65-Pad2): track 7.47 -> 11.8 mm
- net Net-(RL63-Pad2): track 11.8 -> 7.58 mm
Other:
- board size 324.8 x 186 mm -> 315.2 x 186 mm
