File: switch-plate/switch-plate.kicad_pcb (KiCad board)
At the start: 2 copper layers, 303.2 x 124.7 mm, 91 parts

Commit message: Add border to switch plate
A  Footprints.pretty/MountingHole_1.7mm_M1.6_Pad.kicad_mod
M  Footprints.pretty/MountingHole_2.2mm_M2_ISO7380_Pad.kicad_mod
M  placek.py
M  switch-plate/switch-plate.kicad_pcb
M  switch-plate/switch-plate.kicad_sch
Parts:
- H1, H10, H11, H12, H13, H14, H15, H16, H17, H2, H3, H4, H5, H6, H7, H8, H9: footprint MyFootprints:MountingHole_2.2mm_M2_ISO7380_Pad -> MyFootprints:MountingHole_1.7mm_M1.6_Pad

Commit message: Add wrist support plate and remove 2 keys
A  Footprints.pretty/Keychron_Optical_Switch_1.75u.kicad_mod
A  drawborderk.py
M  keychron-optical-keyboard.kicad_pcb
M  keychron-optical-keyboard.kicad_prl
M  keychron-optical-keyboard.kicad_pro
M  keychron-optical-keyboard.kicad_sch
M  placek.py
M  switch-plate/switch-plate.kicad_pcb
M  switch-plate/switch-plate.kicad_sch
A  wrist-support/.gitignore
A  wrist-support/fp-lib-table
A  wrist-support/sym-lib-table
A  wrist-support/wrist-support.kicad_pcb
A  wrist-support/wrist-support.kicad_prl
A  wrist-support/wrist-support.kicad_pro
A  wrist-support/wrist-support.kicad_sch
Parts:
- removed S73, S74: SwitchCutout, MyFootprints:Switch_Cutout
- moved S59 280.9 mm to (14.2, 76.0)
- moved S65 29.7 mm to (137.8, 76.0), turned to 0 degrees
- moved S66 29.7 mm to (162.5, 92.5), turned to 110 degrees
- moved S63 23.3 mm to (94.0, 81.0), turned to -16 degrees
- moved S64 22.2 mm to (113.0, 92.5), turned to 70 degrees
- moved S68 21.0 mm to (199.5, 76.0), turned to 0 degrees
- moved S67 20.2 mm to (179.1, 81.0), turned to 16 degrees
- moved S60 19.0 mm to (33.2, 76.0)
- moved S61 19.0 mm to (52.2, 76.0)
- moved S62 19.0 mm to (71.2, 76.0)
- moved S69 19.0 mm to (218.5, 76.0)
- moved S70 19.0 mm to (237.5, 76.0)
- moved S71 19.0 mm to (256.5, 76.0)
- moved S72 19.0 mm to (275.5, 76.0)
- moved H12 9.50 mm to (294.5, 48.1)
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Other:
- board size 303.2 x 124.7 mm -> 293.8 x 124.7 mm
