File: switch-plate/switch-plate.kicad_sch (KiCad schematic)
At the start: 91 parts

Commit message: Add border to switch plate
A  Footprints.pretty/MountingHole_1.7mm_M1.6_Pad.kicad_mod
M  Footprints.pretty/MountingHole_2.2mm_M2_ISO7380_Pad.kicad_mod
M  placek.py
M  switch-plate/switch-plate.kicad_pcb
M  switch-plate/switch-plate.kicad_sch
Parts:
- H1, H10, H11, H12, H13, H14, H15, H16, H17, H2, H3, H4, H5, H6, H7, H8, H9: footprint MyFootprints:MountingHole_2.2mm_M2_ISO7380_Pad -> MyFootprints:MountingHole_1.7mm_M1.6_Pad

Commit message: Add wrist support plate and remove 2 keys
A  Footprints.pretty/Keychron_Optical_Switch_1.75u.kicad_mod
A  drawborderk.py
M  keychron-optical-keyboard.kicad_pcb
M  keychron-optical-keyboard.kicad_prl
M  keychron-optical-keyboard.kicad_pro
M  keychron-optical-keyboard.kicad_sch
M  placek.py
M  switch-plate/switch-plate.kicad_pcb
M  switch-plate/switch-plate.kicad_sch
A  wrist-support/.gitignore
A  wrist-support/fp-lib-table
A  wrist-support/sym-lib-table
A  wrist-support/wrist-support.kicad_pcb
A  wrist-support/wrist-support.kicad_prl
A  wrist-support/wrist-support.kicad_pro
A  wrist-support/wrist-support.kicad_sch
Parts:
- removed S59, S74: SwitchCutout, MyFootprints:Switch_Cutout, symbol MySym:SwitchCutout
- renumbered S60 to S59, S61 to S60, S62 to S61, S63 to S62, S64 to S63, S65 to S64, S66 to S65, S67 to S66, S68 to S67, S69 to S68, S70 to S69, S71 to S70, S72 to S71, S73 to S72
Changed lines of the file:
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@@
   (symbol (lib_id "MySym:SwitchCutout") (at 133.35 76.2 0) (unit 1)
     (in_bom yes) (on_board yes) (fields_autoplaced)
-    (property "Reference" "S71" (id 0) (at 135.3312 75.3653 0)
+    (property "Reference" "S70" (id 0) (at 135.3312 75.3653 0)
       (effects (font (size 1.27 1.27)) (justify left))
     )
@@
   (symbol (lib_id "MySym:SwitchCutout") (at 64.77 76.2 0) (unit 1)
     (in_bom yes) (on_board yes) (fields_autoplaced)
-    (property "Reference" "S62" (id 0) (at 66.7512 75.3653 0)
+    (property "Reference" "S61" (id 0) (at 66.7512 75.3653 0)
       (effects (font (size 1.27 1.27)) (justify left))
     )
@@
   (symbol (lib_id "MySym:SwitchCutout") (at 57.15 76.2 0) (unit 1)
     (in_bom yes) (on_board yes) (fields_autoplaced)
-    (property "Reference" "S61" (id 0) (at 59.1312 75.3653 0)
+    (property "Reference" "S60" (id 0) (at 59.1312 75.3653 0)
       (effects (font (size 1.27 1.27)) (justify left))
     )
@@
     )
   )
-  (symbol (lib_id "MySym:SwitchCutout") (at 156.21 76.2 0) (unit 1)
-    (in_bom yes) (on_board yes) (fields_autoplaced)
-    (property "Reference" "S74" (id 0) (at 158.1912 75.3653 0)
-      (effects (font (size 1.27 1.27)) (justify left))
-    )
-    (property "Value" "SwitchCutout" (id 1) (at 158.1912 77.9022 0)
-      (effects (font (size 1.27 1.27)) (justify left))
-    )
-    (property "Footprint" "MyFootprints:Switch_Cutout" (id 2) (at 156.21 76.2 0)
-      (effects (font (size 1.27 1.27)) hide)
-    )
-    (property "Datasheet" "" (id 3) (at 156.21 76.2 0)
-      (effects (font (size 1.27 1.27)) hide)
-    )
-  )
   (symbol (lib_id "MySym:SwitchCutout") (at 95.25 60.96 0) (unit 1)
     (in_bom yes) (on_board yes) (fields_autoplaced)
@@
   (symbol (lib_id "MySym:SwitchCutout") (at 87.63 76.2 0) (unit 1)
     (in_bom yes) (on_board yes) (fields_autoplaced)
-    (property "Reference" "S65" (id 0) (at 89.6112 75.3653 0)
+    (property "Reference" "S64" (id 0) (at 89.6112 75.3653 0)
       (effects (font (size 1.27 1.27)) (justify left))
     )
@@
   (symbol (lib_id "MySym:SwitchCutout") (at 140.97 76.2 0) (unit 1)
     (in_bom yes) (on_board yes) (fields_autoplaced)
-    (property "Reference" "S72" (id 0) (at 142.9512 75.3653 0)
+    (property "Reference" "S71" (id 0) (at 142.9512 75.3653 0)
       (effects (font (size 1.27 1.27)) (justify left))
     )
@@
   (symbol (lib_id "MySym:SwitchCutout") (at 80.01 76.2 0) (unit 1)
     (in_bom yes) (on_board yes) (fields_autoplaced)
-    (property "Reference" "S64" (id 0) (at 81.9912 75.3653 0)
+    (property "Reference" "S63" (id 0) (at 81.9912 75.3653 0)
       (effects (font (size 1.27 1.27)) (justify left))
     )
@@
     )
   )
-  (symbol (lib_id "MySym:SwitchCutout") (at 156.21 68.58 0) (unit 1)
-    (in_bom yes) (on_board yes) (fields_autoplaced)
-    (property "Reference" "S59" (id 0) (at 158.1912 67.7453 0)
-      (effects (font (size 1.27 1.27)) (justify left))
-    )
-    (property "Value" "SwitchCutout" (id 1) (at 158.1912 70.2822 0)
-      (effects (font (size 1.27 1.27)) (justify left))
-    )
-    (property "Footprint" "MyFootprints:Switch_Cutout" (id 2) (at 156.21 68.58 0)
-      (effects (font (size 1.27 1.27)) hide)
-    )
-    (property "Datasheet" "" (id 3) (at 156.21 68.58 0)
-      (effects (font (size 1.27 1.27)) hide)
-    )
-  )
   (symbol (lib_id "Mechanical:MountingHole") (at 49.53 116.84 0) (unit 1)
     (in_bom yes) (on_board yes) (fields_autoplaced)
@@
   (symbol (lib_id "MySym:SwitchCutout") (at 118.11 76.2 0) (unit 1)
     (in_bom yes) (on_board yes) (fields_autoplaced)
-    (property "Reference" "S69" (id 0) (at 120.0912 75.3653 0)
+    (property "Reference" "S68" (id 0) (at 120.0912 75.3653 0)
       (effects (font (size 1.27 1.27)) (justify left))
     )
@@
   (symbol (lib_id "MySym:SwitchCutout") (at 110.49 76.2 0) (unit 1)
     (in_bom yes) (on_board yes) (fields_autoplaced)
-    (property "Reference" "S68" (id 0) (at 112.4712 75.3653 0)
+    (property "Reference" "S67" (id 0) (at 112.4712 75.3653 0)
       (effects (font (size 1.27 1.27)) (justify left))
     )
@@
   (symbol (lib_id "MySym:SwitchCutout") (at 72.39 76.2 0) (unit 1)
     (in_bom yes) (on_board yes) (fields_autoplaced)
-    (property "Reference" "S63" (id 0) (at 74.3712 75.3653 0)
+    (property "Reference" "S62" (id 0) (at 74.3712 75.3653 0)
       (effects (font (size 1.27 1.27)) (justify left))
     )
@@
   (symbol (lib_id "MySym:SwitchCutout") (at 95.25 76.2 0) (unit 1)
     (in_bom yes) (on_board yes) (fields_autoplaced)
-    (property "Reference" "S66" (id 0) (at 97.2312 75.3653 0)
+    (property "Reference" "S65" (id 0) (at 97.2312 75.3653 0)
       (effects (font (size 1.27 1.27)) (justify left))
     )
@@
   (symbol (lib_id "MySym:SwitchCutout") (at 102.87 76.2 0) (unit 1)
     (in_bom yes) (on_board yes) (fields_autoplaced)
-    (property "Reference" "S67" (id 0) (at 104.8512 75.3653 0)
+    (property "Reference" "S66" (id 0) (at 104.8512 75.3653 0)
       (effects (font (size 1.27 1.27)) (justify left))
     )
@@
   (symbol (lib_id "MySym:SwitchCutout") (at 148.59 76.2 0) (unit 1)
     (in_bom yes) (on_board yes) (fields_autoplaced)
-    (property "Reference" "S73" (id 0) (at 150.5712 75.3653 0)
+    (property "Reference" "S72" (id 0) (at 150.5712 75.3653 0)
       (effects (font (size 1.27 1.27)) (justify left))
     )
@@
   (symbol (lib_id "MySym:SwitchCutout") (at 125.73 76.2 0) (unit 1)
     (in_bom yes) (on_board yes) (fields_autoplaced)
-    (property "Reference" "S70" (id 0) (at 127.7112 75.3653 0)
+    (property "Reference" "S69" (id 0) (at 127.7112 75.3653 0)
       (effects (font (size 1.27 1.27)) (justify left))
     )
@@
   (symbol (lib_id "MySym:SwitchCutout") (at 49.53 76.2 0) (unit 1)
     (in_bom yes) (on_board yes) (fields_autoplaced)
-    (property "Reference" "S60" (id 0) (at 51.5112 75.3653 0)
+    (property "Reference" "S59" (id 0) (at 51.5112 75.3653 0)
       (effects (font (size 1.27 1.27)) (justify left))
     )
@@
       (reference "S58") (unit 1) (value "SwitchCutout") (footprint "MyFootprints:Switch_Cutout")
     )
-    (path "/69740096-6fd1-4533-82e3-8d507a94b0a5"
+    (path "/f4eb0d3b-6319-4ca1-a028-0a3b793d8d21"
       (reference "S59") (unit 1) (value "SwitchCutout") (footprint "MyFootprints:Switch_Cutout")
     )
-    (path "/f4eb0d3b-6319-4ca1-a028-0a3b793d8d21"
+    (path "/225bb43e-606f-438b-94dd-a50ce1d7d588"
       (reference "S60") (unit 1) (value "SwitchCutout") (footprint "MyFootprints:Switch_Cutout")
     )
-    (path "/225bb43e-606f-438b-94dd-a50ce1d7d588"
+    (path "/0f47508f-9529-4042-be16-cbcda67a8e3a"
       (reference "S61") (unit 1) (value "SwitchCutout") (footprint "MyFootprints:Switch_Cutout")
     )
-    (path "/0f47508f-9529-4042-be16-cbcda67a8e3a"
+    (path "/8ca17128-6a67-43aa-966d-c5b8613f6418"
       (reference "S62") (unit 1) (value "SwitchCutout") (footprint "MyFootprints:Switch_Cutout")
     )
-    (path "/8ca17128-6a67-43aa-966d-c5b8613f6418"
+    (path "/69078fbe-d33c-46a2-8ca4-c2e700b7da95"
       (reference "S63") (unit 1) (value "SwitchCutout") (footprint "MyFootprints:Switch_Cutout")
     )
-    (path "/69078fbe-d33c-46a2-8ca4-c2e700b7da95"
+    (path "/42e59d30-94b1-494c-b122-12d85ddc3ec5"
       (reference "S64") (unit 1) (value "SwitchCutout") (footprint "MyFootprints:Switch_Cutout")
     )
-    (path "/42e59d30-94b1-494c-b122-12d85ddc3ec5"
+    (path "/ab8034eb-5f85-4c17-a8e4-7675821c6936"
       (reference "S65") (unit 1) (value "SwitchCutout") (footprint "MyFootprints:Switch_Cutout")
     )
-    (path "/ab8034eb-5f85-4c17-a8e4-7675821c6936"
+    (path "/c43f1eb4-5ca1-4855-afea-46c7c54b159f"
       (reference "S66") (unit 1) (value "SwitchCutout") (footprint "MyFootprints:Switch_Cutout")
     )
-    (path "/c43f1eb4-5ca1-4855-afea-46c7c54b159f"
+    (path "/7c827d7d-d8fb-4735-96ba-6f67823a1df4"
       (reference "S67") (unit 1) (value "SwitchCutout") (footprint "MyFootprints:Switch_Cutout")
     )
-    (path "/7c827d7d-d8fb-4735-96ba-6f67823a1df4"
+    (path "/6c9666e5-d4b9-427c-bdf1-7ac4d2700f1c"
       (reference "S68") (unit 1) (value "SwitchCutout") (footprint "MyFootprints:Switch_Cutout")
     )
-    (path "/6c9666e5-d4b9-427c-bdf1-7ac4d2700f1c"
+    (path "/e6fec955-8f87-47ea-839c-572d8fe1475f"
       (reference "S69") (unit 1) (value "SwitchCutout") (footprint "MyFootprints:Switch_Cutout")
     )
-    (path "/e6fec955-8f87-47ea-839c-572d8fe1475f"
+    (path "/0ce1d7e4-4b92-4ffd-b41c-5dc024c8f50f"
       (reference "S70") (unit 1) (value "SwitchCutout") (footprint "MyFootprints:Switch_Cutout")
     )
-    (path "/0ce1d7e4-4b92-4ffd-b41c-5dc024c8f50f"
+    (path "/46e09b4d-d91a-4c42-a6ca-5e620516cf71"
       (reference "S71") (unit 1) (value "SwitchCutout") (footprint "MyFootprints:Switch_Cutout")
     )
-    (path "/46e09b4d-d91a-4c42-a6ca-5e620516cf71"
+    (path "/c7f6ba1a-50de-4c28-b4f5-80fb11bec5ed"
       (reference "S72") (unit 1) (value "SwitchCutout") (footprint "MyFootprints:Switch_Cutout")
     )
-    (path "/c7f6ba1a-50de-4c28-b4f5-80fb11bec5ed"
-      (reference "S73") (unit 1) (value "SwitchCutout") (footprint "MyFootprints:Switch_Cutout")
-    )
-    (path "/36cfd324-438d-4d41-be23-0359257e67b8"
-      (reference "S74") (unit 1) (value "SwitchCutout") (footprint "MyFootprints:Switch_Cutout")
-    )
-  )
+  )
